File: AislacionUSB/USBCableIsolatorCircuit.kicad_pcb (KiCad board)
At the start: 2 copper layers, 57.4 x 45 mm, 67 parts, among them CON1 BARREL_JACK, J1 MICRO_USB, J2 IN_VCC, P1 USB_A, U1 PRTR5V0U2X, U2 ADUM5000, U3 7805, U4 PRTR5V0U2X, U5 ADUM4160

Commit message: Se actualizo la rev del PCB y se actualizaron los gerber
Parts:
- D2: value (none) -> D_Schottky
Connections:
- H1 pad 1: (no net) -> Net-(H1-Pad1)
- H2 pad 1: (no net) -> Net-(H2-Pad1)
- H3 pad 1: (no net) -> Net-(H3-Pad1)
Other:
- board text added: "CESE - Aislacion USB Diseño de Circuitos Impresos Marcos Darino - REV01"
- board text added: "REV01"
- board text removed: "CESE - Aislacion USB Diseño de Circuitos Impresos Marcos Darino - REV00"
- board text removed: "REV00"
Changed lines of the file:
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@@
     (zones 0)
     (modules 67)
-    (nets 44)
+    (nets 47)
   )
   (page A4)
@@
     (title "Aislador USB para uso industrial")
     (date 24/7/2016)
-    (rev REV00)
+    (rev REV01)
     (comment 1 "Autor: Marcos Darino")
     (comment 2 "Licencia:  'doc/LICENCIA.txt'")
@@
     (visible_elements 7FFEFFFF)
     (pcbplotparams
-      (layerselection 0x011f0_80000001)
+      (layerselection 0x031f0_80000001)
       (usegerberextensions false)
       (excludeedgelayer true)
@@
   (net 42 "Net-(U2-Pad11)")
   (net 43 "Net-(U2-Pad12)")
+  (net 44 "Net-(H1-Pad1)")
+  (net 45 "Net-(H2-Pad1)")
+  (net 46 "Net-(H3-Pad1)")
   (net_class Default "Esta es la clase de red por defecto."
     (clearance 0.254)
@@
     (add_net "Net-(FB3-Pad2)")
     (add_net "Net-(FB4-Pad1)")
+    (add_net "Net-(H1-Pad1)")
+    (add_net "Net-(H2-Pad1)")
+    (add_net "Net-(H3-Pad1)")
     (add_net "Net-(J1-Pad2)")
     (add_net "Net-(J1-Pad3)")
@@
       (effects (font (size 0.7112 0.4572) (thickness 0.1143)))
     )
-    (fp_text value "" (at 0.3 -3.85 270) (layer F.Fab)
+    (fp_text value D_Schottky (at 0.3 -3.85 270) (layer F.Fab)
       (effects (font (size 0.762 0.762) (thickness 0.127)))
     )
@@
     (fp_circle (center 0 0) (end 2.35 0) (layer Cmts.User) (width 0.15))
     (fp_circle (center 0 0) (end 2.6 0) (layer F.CrtYd) (width 0.05))
-    (pad 1 thru_hole circle (at 0 0) (size 4.7 4.7) (drill 2.7) (layers *.Cu *.Mask F.SilkS))
+    (pad 1 thru_hole circle (at 0 0) (size 4.7 4.7) (drill 2.7) (layers *.Cu *.Mask F.SilkS)
+      (net 44 "Net-(H1-Pad1)"))
   )
   (module AislacionUSB:MountingHole_2.7mm_M2.5_DIN965_Pad (layer F.Cu)
@@
     (fp_circle (center 0 0) (end 2.35 0) (layer Cmts.User) (width 0.15))
     (fp_circle (center 0 0) (end 2.6 0) (layer F.CrtYd) (width 0.05))
-    (pad 1 thru_hole circle (at 0 0) (size 4.7 4.7) (drill 2.7) (layers *.Cu *.Mask F.SilkS))
+    (pad 1 thru_hole circle (at 0 0) (size 4.7 4.7) (drill 2.7) (layers *.Cu *.Mask F.SilkS)
+      (net 45 "Net-(H2-Pad1)"))
   )
   (module AislacionUSB:MountingHole_2.7mm_M2.5_DIN965_Pad (layer F.Cu)
@@
     (fp_circle (center 0 0) (end 2.35 0) (layer Cmts.User) (width 0.15))
     (fp_circle (center 0 0) (end 2.6 0) (layer F.CrtYd) (width 0.05))
-    (pad 1 thru_hole circle (at 0 0) (size 4.7 4.7) (drill 2.7) (layers *.Cu *.Mask F.SilkS))
+    (pad 1 thru_hole circle (at 0 0) (size 4.7 4.7) (drill 2.7) (layers *.Cu *.Mask F.SilkS)
+      (net 46 "Net-(H3-Pad1)"))
   )
   (module AislacionUSB:SRF2012-HandSoldering (layer F.Cu)
@@
     (effects (font (size 1.5 1.5) (thickness 0.375)))
   )
-  (gr_text "CESE  - Aislacion USB\nDiseño de Circuitos Impresos\nMarcos Darino - REV00" (at 131.064 108.204 90) (layer B.SilkS)
+  (gr_text "CESE  - Aislacion USB\nDiseño de Circuitos Impresos\nMarcos Darino - REV01" (at 131.064 108.204 90) (layer B.SilkS)
     (effects (font (size 1.5 1.03) (thickness 0.2575)) (justify mirror))
   )
@@
     (arrow2b (pts (xy 178.308 75.946) (xy 178.894421 77.072504)))
   )
-  (gr_text REV00 (at 165.608 111.633 90) (layer B.Cu)
+  (gr_text REV01 (at 165.608 111.633 90) (layer B.Cu)
     (effects (font (size 1.5 1.5) (thickness 0.375)) (justify mirror))
   )
